Commit message: mujoco

File: src/control_pkg/ros2_control_config/control.ros2_control.xacro (robot description, xacro)
@@ -3,7 +3,8 @@
     <ros2_control name="Pino" type="system">
         <hardware>
-          <plugin>mock_components/GenericSystem</plugin>
+          <!-- <plugin>mock_components/GenericSystem</plugin>
           <param name="mock_sensor_commands">true</param>
-          <param name="position_state_following_offset">0.0</param>
+          <param name="position_state_following_offset">0.0</param> -->
+          <plugin>mujoco_ros2_control/MujocoSystemInterface</plugin>
         </hardware>
         <joint name="fr_hip_joint">

File: src/descrip_pino/urdf/Pino.urdf (robot description, URDF)
Before this commit: robot dog, 13 links, 12 joints
Links:
- link base_link: geometry collision mesh filename=package://descrip_pino/urdf/meshes/base_link.stl; visual mesh filename=package://descrip_pino/urdf/meshes/base_link.stl
- link bl_hip_Link: geometry collision mesh filename=package://descrip_pino/urdf/meshes/bl_hip_Link.stl; visual mesh filename=package://descrip_pino/urdf/meshes/bl_hip_Link.stl
- link bl_knee_Link: geometry collision mesh filename=package://descrip_pino/urdf/meshes/bl_knee_Link.stl; visual mesh filename=package://descrip_pino/urdf/meshes/bl_knee_Link.stl
- link bl_thigh_Link: geometry collision mesh filename=package://descrip_pino/urdf/meshes/bl_thigh_Link.stl; visual mesh filename=package://descrip_pino/urdf/meshes/bl_thigh_Link.stl
- link br_hip_Link: geometry collision mesh filename=package://descrip_pino/urdf/meshes/br_hip_Link.stl; visual mesh filename=package://descrip_pino/urdf/meshes/br_hip_Link.stl
- link br_knee_Link: geometry collision mesh filename=package://descrip_pino/urdf/meshes/br_knee_Link.stl; visual mesh filename=package://descrip_pino/urdf/meshes/br_knee_Link.stl
- link br_thigh_Link: geometry collision mesh filename=package://descrip_pino/urdf/meshes/br_thigh_Link.stl; visual mesh filename=package://descrip_pino/urdf/meshes/br_thigh_Link.stl
- link fl_hip_Link: geometry collision mesh filename=package://descrip_pino/urdf/meshes/fl_hip_Link.stl; visual mesh filename=package://descrip_pino/urdf/meshes/fl_hip_Link.stl
- link fl_knee_Link: geometry collision mesh filename=package://descrip_pino/urdf/meshes/fl_knee_Link.stl; visual mesh filename=package://descrip_pino/urdf/meshes/fl_knee_Link.stl
- link fl_thigh_Link: geometry collision mesh filename=package://descrip_pino/urdf/meshes/fl_thigh_Link.stl; visual mesh filename=package://descrip_pino/urdf/meshes/fl_thigh_Link.stl
- link fr_hip_Link: geometry collision mesh filename=package://descrip_pino/urdf/meshes/fr_hip_Link.stl; visual mesh filename=package://descrip_pino/urdf/meshes/fr_hip_Link.stl
- link fr_knee_Link: geometry collision mesh filename=package://descrip_pino/urdf/meshes/fr_knee_Link.stl; visual mesh filename=package://descrip_pino/urdf/meshes/fr_knee_Link.stl
- link fr_thigh_Link: geometry collision mesh filename=package://descrip_pino/urdf/meshes/fr_thigh_Link.stl; visual mesh filename=package://descrip_pino/urdf/meshes/fr_thigh_Link.stl

Commit message: update

File: src/control_pkg/ros2_control_config/control.ros2_control.xacro (robot description, xacro)
@@ -20,5 +20,4 @@
             <param name="angular_velocity_mjcf_suffix">_gyro</param>
             <param name="linear_acceleration_mjcf_suffix">_accel</param>
-            <param name="topic_name">/imu/data</param>
             <state_interface name="orientation.x"/>
             <state_interface name="orientation.y"/>

File: src/descrip_pino/urdf/Pino.urdf (robot description, URDF)
Before this commit: robot dog, 13 links, 12 joints
Links:
- link base_link: mass 3.79635843826293 -> 4.5
- link bl_hip_Link: mass 1.22881684709264 -> 0.6
- link br_hip_Link: mass 1.2288141630314 -> 0.6
- link fl_hip_Link: mass 1.22881742389137 -> 0.6
- link fr_hip_Link: mass 1.22881616014246 -> 0.6
